Commit message: newcomputer

File: hrwros_ws/src/hrwros_week2/urdf/hrwros_assignment1.xacro (robot description, xacro)
@@ -20,4 +20,5 @@
   <xacro:include filename="$(find hrwros_support)/urdf/bin/bin.urdf.xacro"/>
   <xacro:bin_urdf prefix="bin_1_"/>
+  <xacro:bin_urdf prefix="bin_2_"/>
   <!-- Joints -->
   <joint name="world_interface_to_world" type="fixed">
@@ -72,9 +73,8 @@
   </joint>
   <!-- Add your solution to assignment 1 here -->
-  <xacro:bin_urdf prefix="bin_2_"/>
   <joint name="bin_2_joint" type="fixed">
     <parent link="world_interface" />
     <child link="bin_2_base_link" />
-    <origin xyz="3 2 0" rpy="0 0 0" />
+    <origin xyz="3 2 0" rpy="0 0 0"/>
   </joint>
 </robot>

File: hrwros_ws/src/hrwros_week2/urdf/hrwros_assignment2.xacro (robot description, xacro)
@@ -72,11 +72,11 @@
   </joint>
   <!-- Add your solution to assignment 2 here -->
-<link name="sphere_link">
+  <link name="sphere_link">
     <visual>
-      <origin xyz="0 0 0" />
+      <origin xyz="0 0 0.4" />
       <geometry>
-        <sphere radius ="0.4"/>
+        <sphere radius="0.4" />
       </geometry>
-      <material name="green">
+      <material name="sphere_color">
         <color rgba="0 1 0 1"/>
       </material>
@@ -85,6 +85,6 @@
   <joint name="sphere_joint" type="fixed">
     <parent link="world_interface" />
-    <child link="sphere_link" />
-    <origin xyz="6 -5 0" />
-  </joint
+    <child link="sphere_link"/>
+    <origin xyz="5 -6 0" />
+  </joint>
 </robot>

File: hrwros_ws/src/hrwros_week2/urdf/hrwros_assignment3.urdf (robot description, URDF)
Before this commit: robot robot, 29 links, 29 joints
Links:
- link vacuum_gripper1_suction_cup: mass None -> 0.00001; geometry collision box size=0.001 0.001 0.001; visual box size=0.001 0.001 0.001
Joints:
- removed joint robot2-robot2_fanuc_lrmate200ic
- added joint robot2-robot2_pedestal_joint: type fixed, parent robot2_pedestal_link, child robot2_base_link, origin xyz=0 0 0.6 rpy=0 0 1.57079632679
- joint vacuum_gripper1_joint: origin xyz=0 0 0.080 rpy=0 0 0 -> xyz=0 0 0.01 rpy=0 0 0

File: hrwros_ws/src/hrwros_week2/urdf/hrwros_assignment3.xacro (robot description, xacro)
@@ -66,5 +66,5 @@
   <!-- Update the below block for assignment 3 here -->
   <xacro:include filename="$(find hrwros_week2)/urdf/robot/lrmate200ic_macro.xacro"/>
-  <xacro:ur5_robot prefix="robot2_" joint_limited="true"/>
+  <xacro:fanuc_lrmate200ic prefix="robot2_" joint_limited="true"/>
   <joint name="robot2-robot2_pedestal_joint" type="fixed">
     <parent link="robot2_pedestal_link" />
